Commit message: some changes

File: ROS2_foxy/wheebbot_ws/src/WheeBBot/description/urdf/wheebbot.urdf.xacro (robot description, xacro)
@@ -1,34 +1,5 @@
 <?xml version="1.0"?>
 <robot name="wheebbot" xmlns:xacro="http://www.ros.org/wiki/xacro">
-    <!--%%%%%%%%%%%%%%%% CONSTANTS %%%%%%%%%%%%%%%%-->
-    <xacro:property name="PI" value="3.1415926535897931"/>
-    <xacro:property name="width" value="0.2" />
-    <xacro:property name="bodylen" value="0.6" />
-    <!--%%%%%%%%%%%%%%%% IMPORTING ALL GAZEBO CUSTOMIZATION ELEMENTS %%%%%%%%%%%%%%%%-->
-    <xacro:macro name="leg" params="prefix reflect">
-        <link name="${prefix}_leg">
-            <visual>
-                <geometry>
-                    <box size="${leglen} 0.1 0.2"/>
-                </geometry>
-                <origin xyz="0 0 -${leglen/2}" rpy="0 ${pi/2} 0"/>
-                <material name="white"/>
-            </visual>
-           <collision>
-               <geometry>
-                   <box size="${leglen} 0.1 0.2"/>
-               </geometry>
-               <origin xyz="0 0 -${leglen/2}" rpy="0 ${pi/2} 0"/>
-           </collision>
-           <xacro:default_inertial mass="10"/>
-       </link>
-       <joint name="base_to_${prefix}_leg" type="fixed">
-           <parent link="base_link"/>
-           <child link="${prefix}_leg"/>
-           <origin xyz="0 ${reflect*(width+.02)} 0.25" />
-       </joint>
-       <!-- A bunch of stuff cut -->
-   </xacro:macro>
-   <xacro:leg prefix="right" reflect="1" />
-   <xacro:leg prefix="left" reflect="-1" />
+  <!-- Included URDF/XACRO Files -->
+  <xacro:include filename="$(find wheebbot)/description/urdf/materials.urdf.xacro" />
 </robot>
