Commit message: URDF writing and rviz test

File: ROS2_foxy/wheebbot_ws/src/wheebbot/description/urdf/macros.urdf.xacro (robot description, xacro)
@@ -1,9 +1,23 @@
 <?xml version="1.0"?>
 <robot name="wheebbot" xmlns:xacro="http://www.ros.org/wiki/xacro">
-    <!-- Macro for computing the moments of inertia of a uniform box -->
-    <xacro:macro name="box_inertia" params="l_x l_y l_z mass">
-    <inertia ixx="${1.0/12.0 * mass * (l_y*l_y + l_z*l_z)}" ixy="0.0" ixz="0.0"
-      iyy="${1.0/12.0 * mass * (l_x*l_x + l_z*l_z)}" iyz="0.0"
-      izz="${1.0/12.0 * mass * (l_x*l_x + l_y*l_y)}" />
-    </xacro:macro>
+    <!-- Macro for the inertia tags of a uniform box -->
+  <xacro:macro name="box_inertia" params="mass l_x l_y l_z *origin">
+    <inertial>
+      <xacro:insert_block name="origin" />
+      <mass value="${mass}" />
+      <inertia ixx="${1.0/12.0 * mass * (l_y*l_y + l_z*l_z)}" ixy="0.0" ixz="0.0"
+          iyy="${1.0/12.0 * mass * (l_x*l_x + l_z*l_z)}" iyz="0.0"
+          izz="${1.0/12.0 * mass * (l_x*l_x + l_y*l_y)}" />
+    </inertial>
+  </xacro:macro>
+  <!-- Macro for the inertia tags of a uniform cylinder -->
+  <xacro:macro name="disk_inertia" params="mass radius height *origin">
+    <inertial>
+      <xacro:insert_block name="origin" />
+      <mass value="${mass}" />
+      <inertia ixx="${1.0/12.0 * mass * (3*radius*radius+height*height)}" ixy="0.0" ixz="0.0"
+          iyy="${1.0/12.0 * mass * (3*radius*radius+height*height)}" iyz="0.0"
+          izz="${1.0/2.0 * mass * (radius*radius)}" />
+    </inertial>
+  </xacro:macro>
 </robot>

File: ROS2_foxy/wheebbot_ws/src/wheebbot/description/urdf/parameters.urdf.xacro (robot description, xacro)
@@ -1,9 +1,36 @@
 <?xml version="1.0"?>
 <robot name="wheebbot" xmlns:xacro="http://www.ros.org/wiki/xacro">
-  <xacro:property name="pendulum_mass" value="5.0"/>  <!-- [Kg] -->
-  <xacro:property name="pendulum_length" value="5.0"/>  <!-- [m] -->
-  <xacro:property name="pendulum_CoM_pitch_offset" value="0.0"/>  <!-- [rad] -->
-  <xacro:property name="wheel_mass" value="0.6"/>  <!-- [Kg] -->
-  <xacro:property name="wheel_radius" value="0.06"/>  <!-- [m] -->
-  <xacro:property name="wheels_interax" value="0.4"/>  <!-- [m] -->
+  <!-- Reading some parameters from a YAML config file -->
+  <xacro:property name="yaml_file" value="$(find wheebbot)/config/urdf_params.yaml" />
+  <xacro:property name="props" value="${load_yaml(yaml_file)}"/>
+  <!-- Assigning those parameters to xacro properties -->
+  <xacro:property name="pendulum_mass" value="${props['wheebbot']['pendulum_mass']}" />
+  <xacro:property name="pendulum_length" value="${props['wheebbot']['pendulum_length']}" />
+  <xacro:property name="pendulum_width" value="${props['wheebbot']['pendulum_width']}" />
+  <xacro:property name="pendulum_depth" value="${props['wheebbot']['pendulum_depth']}" />
+  <xacro:property name="pendulum_CoM_pitch_offset" value="${props['wheebbot']['pendulum_CoM_pitch_offset']}" />
+  <xacro:property name="wheel_mass" value="${props['wheebbot']['wheel_mass']}" />
+  <xacro:property name="wheel_radius" value="${props['wheebbot']['wheel_radius']}" />
+  <xacro:property name="wheel_thickness" value="${props['wheebbot']['wheel_thickness']}" />
+  <xacro:property name="wheels_interax" value="${props['wheebbot']['wheels_interax']}" />
+  <xacro:property name="wheel_damping" value="${props['wheebbot']['wheel_damping']}" />
+  <xacro:property name="box_lx" value="${props['wheebbot']['box_lx']}" />
+  <xacro:property name="box_ly" value="${props['wheebbot']['box_ly']}" />
+  <xacro:property name="box_lz" value="${props['wheebbot']['box_lz']}" />
+  <xacro:property name="box_visual_offset_roll" value="${props['wheebbot']['box_visual_offset_roll']}" />
+  <xacro:property name="box_visual_offset_pitch" value="${props['wheebbot']['box_visual_offset_pitch']}" />
+  <xacro:property name="box_visual_offset_yaw" value="${props['wheebbot']['box_visual_offset_yaw']}" />
+  <xacro:property name="leg_length" value="${props['wheebbot']['leg_length']}" />
+  <xacro:property name="leg_extrusion_l_edge" value="${props['wheebbot']['leg_extrusion_l_edge']}" />
+  <xacro:property name="leg_extrusion_l_z" value="${props['wheebbot']['leg_extrusion_l_z']}" />
+  <xacro:property name="leg_pos_wrt_box_back" value="${props['wheebbot']['leg_pos_wrt_box_back']}" />
+  <xacro:property name="fan_edge_length" value="${props['wheebbot']['fan_edge_length']}" />
+  <xacro:property name="fan_vert_footprint" value="${props['wheebbot']['fan_vert_footprint']}" />
+  <xacro:property name="motor_case_l_edge" value="${props['wheebbot']['motor_case_l_edge']}" />
+  <xacro:property name="motor_case_extension" value="${props['wheebbot']['motor_case_extension']}" />
+  <xacro:property name="door_handle_tot_height" value="${props['wheebbot']['door_handle_tot_height']}" />
+  <xacro:property name="door_handle_height2" value="${props['wheebbot']['door_handle_height2']}" />
+  <xacro:property name="door_handle_tot_lenght" value="${props['wheebbot']['door_handle_tot_lenght']}" />
+  <xacro:property name="door_handle_lenght2" value="${props['wheebbot']['door_handle_lenght2']}" />
+  <xacro:property name="door_handle_width" value="${props['wheebbot']['door_handle_width']}" />
 </robot>

File: ROS2_foxy/wheebbot_ws/src/wheebbot/description/urdf/wheebbot.urdf.xacro (robot description, xacro)
@@ -1,50 +1,14 @@
 <?xml version="1.0"?>
 <robot name="wheebbot" xmlns:xacro="http://www.ros.org/wiki/xacro">
-  <!-- Stuff after $ is interpreted by Python -->
-  <xacro:property name="PI" value="${pi}" />
-  <!-- Reading some parameters from YAML config file -->
-  <xacro:property name="yaml_file" value="$(find wheebbot)/config/urdf_params.yaml" />
-  <xacro:property name="props" value="${load_yaml(yaml_file)}"/>
-  <!-- Assigning those parameters to xacro properties -->
-  <xacro:property name="pendulum_mass" value="${props['wheebbot']['pendulum_mass']}" />
-  <xacro:property name="pendulum_length" value="${props['wheebbot']['pendulum_length']}" />
-  <xacro:property name="pendulum_CoM_pitch_offset" value="${props['wheebbot']['pendulum_CoM_pitch_offset']}" />
-  <xacro:property name="wheel_mass" value="${props['wheebbot']['wheel_mass']}" />
-  <xacro:property name="wheel_radius" value="${props['wheebbot']['wheel_radius']}" />
-  <xacro:property name="wheel_thickness" value="${props['wheebbot']['wheel_thickness']}" />
-  <xacro:property name="wheels_interax" value="${props['wheebbot']['wheels_interax']}" />
-  <xacro:property name="wheel_damping" value="${props['wheebbot']['wheel_damping']}" />
-  <xacro:property name="box_lx" value="${props['wheebbot']['box_lx']}" />
-  <xacro:property name="box_ly" value="${props['wheebbot']['box_ly']}" />
-  <xacro:property name="box_lz" value="${props['wheebbot']['box_lz']}" />
-  <xacro:property name="box_visual_offset_roll" value="${props['wheebbot']['box_visual_offset_roll']}" />
-  <xacro:property name="box_visual_offset_pitch" value="${props['wheebbot']['box_visual_offset_pitch']}" />
-  <xacro:property name="box_visual_offset_yaw" value="${props['wheebbot']['box_visual_offset_yaw']}" />
-  <xacro:property name="leg_length" value="${props['wheebbot']['leg_length']}" />
-  <!-- <xacro:include filename="$(find wheebbot)/description/urdf/parameters.urdf.xacro" /> -->
-  <!-- Macro for the inertia tags of a uniform box -->
-  <xacro:macro name="box_inertia" params="mass l_x l_y l_z *origin">
-    <inertial>
-      <xacro:insert_block name="origin" />
-      <mass value="${mass}" />
-      <inertia ixx="${1.0/12.0 * mass * (l_y*l_y + l_z*l_z)}" ixy="0.0" ixz="0.0"
-          iyy="${1.0/12.0 * mass * (l_x*l_x + l_z*l_z)}" iyz="0.0"
-          izz="${1.0/12.0 * mass * (l_x*l_x + l_y*l_y)}" />
-    </inertial>
-  </xacro:macro>
-  <!-- Macro for the inertia tags of a uniform cylinder -->
-  <xacro:macro name="disk_inertia" params="mass radius height *origin">
-    <inertial>
-      <xacro:insert_block name="origin" />
-      <mass value="${mass}" />
-      <inertia ixx="${1.0/12.0 * mass * (3*radius*radius+height*height)}" ixy="0.0" ixz="0.0"
-          iyy="${1.0/12.0 * mass * (3*radius*radius+height*height)}" iyz="0.0"
-          izz="${1.0/2.0 * mass * (radius*radius)}" />
-    </inertial>
-  </xacro:macro>
+  <!-- Including the parameters file -->
+  <xacro:include filename="$(find wheebbot)/description/urdf/parameters.urdf.xacro" />
+  <!-- Including the macros file -->
+  <xacro:include filename="$(find wheebbot)/description/urdf/macros.urdf.xacro" />
+  <link name="base_link">
+  </link>
   <link name="body">
     <!-- body visual -->
     <visual>
-      <origin xyz="0 0 0" rpy="0 0 0" />
+      <origin xyz="0 ${box_ly/2-leg_extrusion_l_edge/2} ${-(box_lz/2-leg_extrusion_l_edge/2)}" rpy="0 0 ${-pi/2}" />
       <geometry>
         <mesh filename="package://wheebbot/description/meshes/full_no_knee_no_wheels.dae" scale="1.0 1.0 1.0" />
@@ -55,29 +19,84 @@
       <origin xyz="0 0 0" rpy="0 0 0"/>
         <geometry>
-          <box size="1 1 1" />
+          <box size="${box_lx} ${box_ly} ${box_lz}" />
+        </geometry>
+    </collision>
+   <!-- top fan collision group-->
+   <!-- fan-->
+    <collision>
+      <origin xyz="0 0 ${(box_lz/2+fan_vert_footprint/2)}" rpy="0 0 0"/>
+        <geometry>
+          <box size="${fan_edge_length} ${fan_edge_length} ${fan_vert_footprint}" />
+        </geometry>
+    </collision>
+    <!-- left door handle-->
+    <collision>
+      <origin xyz="0 ${box_ly/2-door_handle_width/2} ${(box_lz/2+door_handle_height2/2)}" rpy="0 0 0"/>
+        <geometry>
+          <box size="${door_handle_tot_lenght} ${door_handle_width} ${door_handle_height2}" />
+        </geometry>
+    </collision>
+    <collision>
+      <origin xyz="0 ${box_ly/2-door_handle_width/2} ${(box_lz/2+door_handle_height2+(door_handle_tot_height-door_handle_height2)/2)}" rpy="0 0 0"/>
+        <geometry>
+          <box size="${door_handle_lenght2} ${door_handle_width} ${door_handle_tot_height-door_handle_height2}" />
+        </geometry>
+    </collision>
+    <!-- right door handle-->
+    <collision>
+       <origin xyz="0 ${-(box_ly/2-door_handle_width/2)} ${(box_lz/2+door_handle_height2/2)}" rpy="0 0 0"/>
+         <geometry>
+           <box size="${door_handle_tot_lenght} ${door_handle_width} ${door_handle_height2}" />
+         </geometry>
+     </collision>
+     <collision>
+       <origin xyz="0 ${-(box_ly/2-door_handle_width/2)} ${(box_lz/2+door_handle_height2+(door_handle_tot_height-door_handle_height2)/2)}" rpy="0 0 0"/>
+         <geometry>
+           <box size="${door_handle_lenght2} ${door_handle_width} ${door_handle_tot_height-door_handle_height2}" />
+         </geometry>
+     </collision>
+    <!-- back fan collision -->
+    <collision>
+      <origin xyz="${-(box_lx/2+fan_vert_footprint/2)} 0 0" rpy="0 ${-pi/2} 0"/>
+        <geometry>
+          <box size="${fan_edge_length} ${fan_edge_length} ${fan_vert_footprint}" />
         </geometry>
     </collision>
     <!-- left leg -->
     <collision>
-      <origin xyz="0 0 0" rpy="0 0 0"/>
+      <origin xyz="${(leg_pos_wrt_box_back-box_lx/2)} ${box_ly/2-leg_extrusion_l_edge/2} ${-(box_lz/2+leg_length/2)}" rpy="0 0 0"/>
         <geometry>
-          <box size="1 1 1" />
+          <box size="${leg_extrusion_l_edge} ${leg_extrusion_l_edge} ${leg_length}" />
+        </geometry>
+    </collision>
+    <!-- left motor case -->
+    <collision>
+      <origin xyz="${(leg_pos_wrt_box_back-box_lx/2)} ${box_ly/2-motor_case_extension/2} ${-(box_lz/2+leg_length+motor_case_l_edge/2)}" rpy="0 0 0"/>
+        <geometry>
+          <box size="${motor_case_l_edge} ${motor_case_extension} ${motor_case_l_edge}" />
         </geometry>
     </collision>
     <!-- right leg -->
     <collision>
-      <origin xyz="0 0 0" rpy="0 0 0"/>
+      <origin xyz="${(leg_pos_wrt_box_back-box_lx/2)} ${-(box_ly/2-leg_extrusion_l_edge/2)} ${-(box_lz/2+leg_length/2)}" rpy="0 0 0"/>
         <geometry>
-          <box size="1 1 1" />
+          <box size="${leg_extrusion_l_edge} ${leg_extrusion_l_edge} ${leg_length}" />
         </geometry>
     </collision>
-    <xacro:box_inertia mass="${}" lx="${}" ly="${}" lz="${}" >
-      <origin xyz="${}" rpy="${}" />
-    </xacro:box_inertia >
+    <!-- right motor case -->
+    <collision>
+      <origin xyz="${(leg_pos_wrt_box_back-box_lx/2)} ${-(box_ly/2-motor_case_extension/2)} ${-(box_lz/2+leg_length+motor_case_l_edge/2)}" rpy="0 0 0"/>
+        <geometry>
+          <box size="${motor_case_l_edge} ${motor_case_extension} ${motor_case_l_edge}" />
+        </geometry>
+    </collision>
+    <xacro:box_inertia mass="${pendulum_mass}" l_x="${pendulum_depth}" l_y="${pendulum_width}" l_z="${pendulum_length}">
+      <origin xyz="${pendulum_length*sin(pendulum_CoM_pitch_offset)} 0 ${-(box_lz/2+leg_length+motor_case_l_edge/2)+pendulum_length*cos(pendulum_CoM_pitch_offset)}" rpy="0 ${pendulum_CoM_pitch_offset} 0"/>
+    </xacro:box_inertia>
   </link>
   <link name="left_wheel">
     <!-- wheel visual -->
     <visual>
-      <origin xyz="0 0 0" rpy="0 0 0" />
+      <origin xyz="0 0 0" rpy="0 0 ${pi/2}" />
       <geometry>
         <mesh filename="package://wheebbot/description/meshes/wheel_full.dae" scale="1.0 1.0 1.0" />
@@ -85,17 +104,17 @@
     </visual>
     <collision>
-      <origin xyz="0 0 0" rpy="0 0 0"/>
+      <origin xyz="0 0 0" rpy="${pi/2} 0 0"/>
         <geometry>
           <cylinder radius="${wheel_radius}" length="${wheel_thickness}"/>
         </geometry>
     </collision>
-    <xacro:disk_inertia mass="${}" radius="${}" height="${}">
-      <origin xyz="${}" rpy="${}" />
-    </xacro:box_inertia >
+    <xacro:disk_inertia mass="${wheel_mass}" radius="${wheel_radius}" height="${wheel_thickness}">
+      <origin xyz="0 0 0" rpy="${-pi/2} 0 0" />
+    </xacro:disk_inertia>
   </link>
   <link name="right_wheel">
     <!-- wheel visual -->
     <visual>
-      <origin xyz="0 0 0" rpy="0 0 0" />
+      <origin xyz="0 0 0" rpy="0 0 ${-pi/2}" />
       <geometry>
         <mesh filename="package://wheebbot/description/meshes/wheel_full.dae" scale="1.0 1.0 1.0" />
@@ -103,15 +122,20 @@
     </visual>
     <collision>
-      <origin xyz="0 0 0" rpy="0 0 0"/>
+      <origin xyz="0 0 0" rpy="${pi/2} 0 0"/>
         <geometry>
           <cylinder radius="${wheel_radius}" length="${wheel_thickness}"/>
         </geometry>
     </collision>
-    <xacro:disk_inertia mass="${}" radius="${}" height="${}">
-      <origin xyz="${}" rpy="${}" />
-    </xacro:box_inertia >
+    <xacro:disk_inertia mass="${wheel_mass}" radius="${wheel_radius}" height="${wheel_thickness}">
+      <origin xyz="0 0 0" rpy="${-pi/2} 0 0" />
+    </xacro:disk_inertia >
   </link>
+  <joint name="floating_base_joint" type="fixed">
+    <origin xyz="0 0 0" rpy="0 0 0"/>
+    <parent link="base_link"/>
+    <child link="body"/>
+  </joint>
   <joint name="left_wheel_joint" type="continuous">
-    <origin xyz="0 0 0" rpy="0 0 0"/>
+    <origin xyz="0 ${(wheels_interax/2)} ${-(box_lz/2+leg_length+motor_case_l_edge/2)}" rpy="0 0 0"/>
     <parent link="body"/>
     <child link="left_wheel"/>
@@ -121,5 +145,5 @@
   </joint>
   <joint name="right_wheel_joint" type="continuous">
-    <origin xyz="0 0 0" rpy="0 0 0"/>
+    <origin xyz="0 ${-(wheels_interax/2)} ${-(box_lz/2+leg_length+motor_case_l_edge/2)}" rpy="0 0 0"/>
     <parent link="body"/>
     <child link="right_wheel"/>
