Commit message: small changes

File: ROS2_foxy/wheebbot_ws/src/wheebbot/description/urdf/materials.urdf.xacro (robot description, xacro)
@@ -1,27 +1,27 @@
 <?xml version="1.0"?>
-<robot name="wheebbot" xmlns:xacro="http://www.ros.org/wiki/xacro">
-  <material name="Black">
+<robot>
+  <material name="black">
     <color rgba="0.0 0.0 0.0 1.0"/>
   </material>
-  <material name="Blue">
+  <material name="blue">
     <color rgba="0.0 0.0 0.8 1.0"/>
   </material>
-  <material name="Green">
+  <material name="green">
     <color rgba="0.0 0.8 0.0 1.0"/>
   </material>
-  <material name="Gray">
-    <color rgba="0.7 0.7 0.7 1.0"/>
+  <material name="grey">
+    <color rgba="0.2 0.2 0.2 1.0"/>
   </material>
-  <material name="DarkGray">
-    <color rgba="0.3 0.3 0.3 1.0"/>
+  <material name="orange">
+    <color rgba="${255/255} ${108/255} ${10/255} 1.0"/>
   </material>
-  <material name="Red">
+  <material name="brown">
+    <color rgba="${222/255} ${207/255} ${195/255} 1.0"/>
+  </material>
+  <material name="red">
     <color rgba="0.8 0.0 0.0 1.0"/>
   </material>
-  <material name="White">
+  <material name="white">
     <color rgba="1.0 1.0 1.0 1.0"/>
   </material>
-  <material name="Yellow">
-    <color rgba="0.8 0.8 0.0 1.0"/>
-  </material>
 </robot>

File: ROS2_foxy/wheebbot_ws/src/wheebbot/description/urdf/parameters.urdf.xacro (robot description, xacro)
@@ -1,4 +1,4 @@
 <?xml version="1.0"?>
-<robot name="wheebbot" xmlns:xacro="http://www.ros.org/wiki/xacro">
+<robot>
   <!-- Reading some parameters from a YAML config file -->
   <xacro:property name="yaml_file" value="$(find wheebbot)/config/urdf_params.yaml" />

File: ROS2_foxy/wheebbot_ws/src/wheebbot/description/urdf/wheebbot.gazebo.xacro (robot description, xacro)
@@ -1,10 +1,25 @@
 <?xml version="1.0"?>
-<robot name="wheebbot" xmlns:xacro="http://www.ros.org/wiki/xacro">
-    <gazebo reference="LF_FOOT">
-        <!-- Foot contact parameters -->
-        <kp>1000000.0</kp>
-        <kd>100.0</kd>
-        <mu1>0.8</mu1>
-        <mu2>0.8</mu2>
-    </gazebo>
+<robot>
+  <!-- ros_control plugin -->
+  <gazebo>
+    <plugin name="gazebo_ros_joint_state_publisher" filename="libgazebo_ros_joint_state_publisher.so">
+      <update_rate>20</update_rate>
+      <joint_name>left_wheel_joint</joint_name>
+      <joint_name>right_wheel_joint</joint_name>
+    </plugin>
+  </gazebo>
+  <!-- Link1 -->
+  <gazebo reference="link1">
+    <material>Gazebo/Orange</material>
+  </gazebo>
+  <!-- Link2 -->
+  <gazebo reference="right_wheel">
+    <mu1>0.5</mu1>
+    <mu2>0.5</mu2>
+  </gazebo>
+  <!-- Link3 -->
+  <gazebo reference="left_wheel">
+    <mu1>0.5</mu1>
+    <mu2>0.5</mu2>
+  </gazebo>
 </robot>

File: ROS2_foxy/wheebbot_ws/src/wheebbot/description/urdf/wheebbot.urdf.xacro (robot description, xacro)
@@ -5,4 +5,8 @@
   <!-- Including the macros file -->
   <xacro:include filename="$(find wheebbot)/description/urdf/macros.urdf.xacro" />
+  <!-- Including the materials file -->
+  <xacro:include filename="$(find wheebbot)/description/urdf/materials.urdf.xacro" />
+  <!-- Including the gazebo file -->
+  <xacro:include filename="$(find wheebbot)/description/urdf/wheebbot.gazebo.xacro" />
   <link name="base_link">
   </link>
