Commit message: small changes

File: ROS2_foxy/wheebbot_ws/src/wheebbot/description/urdf/wheebbot.gazebo.xacro (robot description, xacro)
@@ -9,14 +9,10 @@
     </plugin>
   </gazebo>
-  <!-- Link1 -->
-  <gazebo reference="link1">
-    <material>Gazebo/Orange</material>
-  </gazebo>
-  <!-- Link2 -->
+  <!-- right wheel -->
   <gazebo reference="right_wheel">
     <mu1>0.5</mu1>
     <mu2>0.5</mu2>
   </gazebo>
-  <!-- Link3 -->
+  <!-- left wheel -->
   <gazebo reference="left_wheel">
     <mu1>0.5</mu1>

File: ROS2_foxy/wheebbot_ws/src/wheebbot/description/urdf/wheebbot.urdf.xacro (robot description, xacro)
@@ -7,5 +7,5 @@
   <!-- Including the materials file -->
   <xacro:include filename="$(find wheebbot)/description/urdf/materials.urdf.xacro" />
-  <!-- Including the gazebo file -->
+  <!-- Including the gazebo related stuff -->
   <xacro:include filename="$(find wheebbot)/description/urdf/wheebbot.gazebo.xacro" />
   <link name="base_link">

Commit message: successfull joint state publisher from gazebo to rviz

File: ROS2_foxy/wheebbot_ws/src/wheebbot/description/urdf/wheebbot.gazebo.xacro (robot description, xacro)
@@ -1,5 +1,5 @@
 <?xml version="1.0"?>
 <robot xmlns:xacro="http://www.ros.org/wiki/xacro">
-  <!-- ros_control plugin -->
+  <!-- joint state publisher (this way gazebo publishes joint states to RViz) -->
   <gazebo>
     <plugin name="gazebo_ros_joint_state_publisher" filename="libgazebo_ros_joint_state_publisher.so">

File: ROS2_foxy/wheebbot_ws/src/wheebbot/description/urdf/wheebbot.urdf.xacro (robot description, xacro)
@@ -136,5 +136,5 @@
   </link>
   <joint name="floating_base_joint" type="fixed">
-    <origin xyz="0 0 0" rpy="0 0 0"/>
+    <origin xyz="0 0 ${(box_lz/2+leg_length+motor_case_l_edge/2+wheel_radius)}" rpy="0 0 0"/>
     <parent link="base_link"/>
     <child link="body"/>
