Commit message: updates

File: ROS2_foxy/wheebbot_ws/src/wheebbot/description/urdf/wheebbot.urdf.xacro (robot description, xacro)
@@ -1,5 +1,130 @@
 <?xml version="1.0"?>
 <robot name="wheebbot" xmlns:xacro="http://www.ros.org/wiki/xacro">
-  <!-- Included URDF/XACRO Files -->
-  <xacro:include filename="$(find wheebbot)/description/urdf/materials.urdf.xacro" />
+  <!-- Stuff after $ is interpreted by Python -->
+  <xacro:property name="PI" value="${pi}" />
+  <!-- Reading some parameters from YAML config file -->
+  <xacro:property name="yaml_file" value="$(find wheebbot)/config/urdf_params.yaml" />
+  <xacro:property name="props" value="${load_yaml(yaml_file)}"/>
+  <!-- Assigning those parameters to xacro properties -->
+  <xacro:property name="pendulum_mass" value="${props['wheebbot']['pendulum_mass']}" />
+  <xacro:property name="pendulum_length" value="${props['wheebbot']['pendulum_length']}" />
+  <xacro:property name="pendulum_CoM_pitch_offset" value="${props['wheebbot']['pendulum_CoM_pitch_offset']}" />
+  <xacro:property name="wheel_mass" value="${props['wheebbot']['wheel_mass']}" />
+  <xacro:property name="wheel_radius" value="${props['wheebbot']['wheel_radius']}" />
+  <xacro:property name="wheel_thickness" value="${props['wheebbot']['wheel_thickness']}" />
+  <xacro:property name="wheels_interax" value="${props['wheebbot']['wheels_interax']}" />
+  <xacro:property name="wheel_damping" value="${props['wheebbot']['wheel_damping']}" />
+  <xacro:property name="box_lx" value="${props['wheebbot']['box_lx']}" />
+  <xacro:property name="box_ly" value="${props['wheebbot']['box_ly']}" />
+  <xacro:property name="box_lz" value="${props['wheebbot']['box_lz']}" />
+  <xacro:property name="box_visual_offset_roll" value="${props['wheebbot']['box_visual_offset_roll']}" />
+  <xacro:property name="box_visual_offset_pitch" value="${props['wheebbot']['box_visual_offset_pitch']}" />
+  <xacro:property name="box_visual_offset_yaw" value="${props['wheebbot']['box_visual_offset_yaw']}" />
+  <xacro:property name="leg_length" value="${props['wheebbot']['leg_length']}" />
+  <!-- <xacro:include filename="$(find wheebbot)/description/urdf/parameters.urdf.xacro" /> -->
+  <!-- Macro for the inertia tags of a uniform box -->
+  <xacro:macro name="box_inertia" params="mass l_x l_y l_z *origin">
+    <inertial>
+      <xacro:insert_block name="origin" />
+      <mass value="${mass}" />
+      <inertia ixx="${1.0/12.0 * mass * (l_y*l_y + l_z*l_z)}" ixy="0.0" ixz="0.0"
+          iyy="${1.0/12.0 * mass * (l_x*l_x + l_z*l_z)}" iyz="0.0"
+          izz="${1.0/12.0 * mass * (l_x*l_x + l_y*l_y)}" />
+    </inertial>
+  </xacro:macro>
+  <!-- Macro for the inertia tags of a uniform cylinder -->
+  <xacro:macro name="disk_inertia" params="mass radius height *origin">
+    <inertial>
+      <xacro:insert_block name="origin" />
+      <mass value="${mass}" />
+      <inertia ixx="${1.0/12.0 * mass * (3*radius*radius+height*height)}" ixy="0.0" ixz="0.0"
+          iyy="${1.0/12.0 * mass * (3*radius*radius+height*height)}" iyz="0.0"
+          izz="${1.0/2.0 * mass * (radius*radius)}" />
+    </inertial>
+  </xacro:macro>
+  <link name="body">
+    <!-- body visual -->
+    <visual>
+      <origin xyz="0 0 0" rpy="0 0 0" />
+      <geometry>
+        <mesh filename="package://wheebbot/description/meshes/full_no_knee_no_wheels.dae" scale="1.0 1.0 1.0" />
+      </geometry>
+    </visual>
+    <!-- box -->
+    <collision>
+      <origin xyz="0 0 0" rpy="0 0 0"/>
+        <geometry>
+          <box size="1 1 1" />
+        </geometry>
+    </collision>
+    <!-- left leg -->
+    <collision>
+      <origin xyz="0 0 0" rpy="0 0 0"/>
+        <geometry>
+          <box size="1 1 1" />
+        </geometry>
+    </collision>
+    <!-- right leg -->
+    <collision>
+      <origin xyz="0 0 0" rpy="0 0 0"/>
+        <geometry>
+          <box size="1 1 1" />
+        </geometry>
+    </collision>
+    <xacro:box_inertia mass="${}" lx="${}" ly="${}" lz="${}" >
+      <origin xyz="${}" rpy="${}" />
+    </xacro:box_inertia >
+  </link>
+  <link name="left_wheel">
+    <!-- wheel visual -->
+    <visual>
+      <origin xyz="0 0 0" rpy="0 0 0" />
+      <geometry>
+        <mesh filename="package://wheebbot/description/meshes/wheel_full.dae" scale="1.0 1.0 1.0" />
+      </geometry>
+    </visual>
+    <collision>
+      <origin xyz="0 0 0" rpy="0 0 0"/>
+        <geometry>
+          <cylinder radius="${wheel_radius}" length="${wheel_thickness}"/>
+        </geometry>
+    </collision>
+    <xacro:disk_inertia mass="${}" radius="${}" height="${}">
+      <origin xyz="${}" rpy="${}" />
+    </xacro:box_inertia >
+  </link>
+  <link name="right_wheel">
+    <!-- wheel visual -->
+    <visual>
+      <origin xyz="0 0 0" rpy="0 0 0" />
+      <geometry>
+        <mesh filename="package://wheebbot/description/meshes/wheel_full.dae" scale="1.0 1.0 1.0" />
+      </geometry>
+    </visual>
+    <collision>
+      <origin xyz="0 0 0" rpy="0 0 0"/>
+        <geometry>
+          <cylinder radius="${wheel_radius}" length="${wheel_thickness}"/>
+        </geometry>
+    </collision>
+    <xacro:disk_inertia mass="${}" radius="${}" height="${}">
+      <origin xyz="${}" rpy="${}" />
+    </xacro:box_inertia >
+  </link>
+  <joint name="left_wheel_joint" type="continuous">
+    <origin xyz="0 0 0" rpy="0 0 0"/>
+    <parent link="body"/>
+    <child link="left_wheel"/>
+    <axis xyz="0 1 0" />
+    <dynamics damping="0.0" friction="0.0"/>
+    <limit effort="30" velocity="100.0" />
+  </joint>
+  <joint name="right_wheel_joint" type="continuous">
+    <origin xyz="0 0 0" rpy="0 0 0"/>
+    <parent link="body"/>
+    <child link="right_wheel"/>
+    <axis xyz="0 1 0" />
+    <dynamics damping="0.0" friction="0.0"/>
+    <limit effort="30" velocity="100.0" />
+  </joint>
 </robot>

Commit message: ignition test and successfull custom world launch

File: ROS2_foxy/wheebbot_ws/src/wheebbot/description/urdf/wheebbot.urdf.xacro (robot description, xacro)
@@ -9,5 +9,5 @@
   <!-- Including the gazebo related stuff -->
   <xacro:include filename="$(find wheebbot)/description/urdf/wheebbot.gazebo.xacro" />
-  <link name="base_link">
+  <link name="aux_link">
   </link>
   <link name="body">
@@ -104,5 +104,5 @@
       <origin xyz="0 0 0" rpy="0 0 ${pi/2}" />
       <geometry>
-        <mesh filename="package://wheebbot/description/meshes/wheel_full.dae" scale="1.0 1.0 1.0" />
+        <mesh filename="package://wheebbot/description/meshes/wheel_black.dae" scale="1.0 1.0 1.0" />
       </geometry>
     </visual>
@@ -122,5 +122,5 @@
       <origin xyz="0 0 0" rpy="0 0 ${-pi/2}" />
       <geometry>
-        <mesh filename="package://wheebbot/description/meshes/wheel_full.dae" scale="1.0 1.0 1.0" />
+        <mesh filename="package://wheebbot/description/meshes/wheel_black.dae" scale="1.0 1.0 1.0" />
       </geometry>
     </visual>
@@ -135,7 +135,7 @@
     </xacro:disk_inertia >
   </link>
-  <joint name="floating_base_joint" type="fixed">
+  <joint name="aux_joint" type="fixed">
     <origin xyz="0 0 ${(box_lz/2+leg_length+motor_case_l_edge/2+wheel_radius)}" rpy="0 0 0"/>
-    <parent link="base_link"/>
+    <parent link="aux_link"/>
     <child link="body"/>
   </joint>
