Commit message: small improvements

File: ROS2_foxy/wheebbot_ws/src/wheebbot/description/urdf/parameters.urdf.xacro (robot description, xacro)
@@ -14,11 +14,20 @@
   <xacro:property name="wheel_thickness" value="${props['wheebbot']['wheel_thickness']}" />
   <xacro:property name="wheels_interax" value="${props['wheebbot']['wheels_interax']}" />
-  <xacro:property name="wheel_damping" value="${props['wheebbot']['wheel_damping']}" />
+  <xacro:property name="wheel_joint_damping" value="${props['wheebbot']['wheel_joint_damping']}" />
+  <xacro:property name="wheel_joint_static_friction" value="${props['wheebbot']['wheel_joint_static_friction']}" />
+  <xacro:property name="wheel_joint_effort_lim" value="${props['wheebbot']['wheel_joint_effort_lim']}" />
+  <xacro:property name="wheel_joint_velocity_lim" value="${props['wheebbot']['wheel_joint_velocity_lim']}" />
+  <xacro:property name="wheel_mu1_gazebo" value="${props['wheebbot']['wheel_mu1_gazebo']}" />
+  <xacro:property name="wheel_mu2_gazebo" value="${props['wheebbot']['wheel_mu2_gazebo']}" />
+  <xacro:property name="wheel_kp_gazebo" value="${props['wheebbot']['wheel_kp_gazebo']}" />
+  <xacro:property name="wheel_kd_gazebo" value="${props['wheebbot']['wheel_kd_gazebo']}" />
+  <xacro:property name="wheel_max_contacts_gazebo" value="${props['wheebbot']['wheel_max_contacts_gazebo']}" />
+  <xacro:property name="body_mu1_gazebo" value="${props['wheebbot']['body_mu1_gazebo']}" />
+  <xacro:property name="body_mu2_gazebo" value="${props['wheebbot']['body_mu2_gazebo']}" />
+  <xacro:property name="body_kp_gazebo" value="${props['wheebbot']['body_kp_gazebo']}" />
+  <xacro:property name="body_kd_gazebo" value="${props['wheebbot']['body_kd_gazebo']}" />
   <xacro:property name="box_lx" value="${props['wheebbot']['box_lx']}" />
   <xacro:property name="box_ly" value="${props['wheebbot']['box_ly']}" />
   <xacro:property name="box_lz" value="${props['wheebbot']['box_lz']}" />
-  <xacro:property name="box_visual_offset_roll" value="${props['wheebbot']['box_visual_offset_roll']}" />
-  <xacro:property name="box_visual_offset_pitch" value="${props['wheebbot']['box_visual_offset_pitch']}" />
-  <xacro:property name="box_visual_offset_yaw" value="${props['wheebbot']['box_visual_offset_yaw']}" />
   <xacro:property name="leg_length" value="${props['wheebbot']['leg_length']}" />
   <xacro:property name="leg_extrusion_l_edge" value="${props['wheebbot']['leg_extrusion_l_edge']}" />

File: ROS2_foxy/wheebbot_ws/src/wheebbot/description/urdf/wheebbot.gazebo.xacro (robot description, xacro)
@@ -11,24 +11,24 @@
   <!-- body -->
   <gazebo reference="body">
-    <mu1>0.3</mu1>
-    <mu2>0.3</mu2>
-    <kp>500000000000000</kp>
-    <kd>1</kd>
+    <mu1>${body_mu1_gazebo}</mu1>
+    <mu2>${body_mu2_gazebo}</mu2>
+    <kp>${body_kp_gazebo}</kp>
+    <kd>${body_kd_gazebo}</kd>
   </gazebo>
   <!-- right wheel -->
   <gazebo reference="right_wheel">
-    <mu1>0.5</mu1>
-    <mu2>0.5</mu2>
-    <kp>500000000000000</kp>
-    <kd>1</kd>
-    <maxContacts>10</maxContacts>
+    <mu1>${wheel_mu1_gazebo}</mu1>
+    <mu2>${wheel_mu2_gazebo}</mu2>
+    <kp>${wheel_kp_gazebo}</kp>
+    <kd>${wheel_kd_gazebo}</kd>
+    <maxContacts>${wheel_max_contacts_gazebo}</maxContacts>
   </gazebo>
   <!-- left wheel -->
   <gazebo reference="left_wheel">
-    <mu1>0.5</mu1>
-    <mu2>0.5</mu2>
-    <kp>500000000000000</kp>
-    <kd>1</kd>
-    <maxContacts>10</maxContacts>
+    <mu1>${wheel_mu1_gazebo}</mu1>
+    <mu2>${wheel_mu2_gazebo}</mu2>
+    <kp>${wheel_kp_gazebo}</kp>
+    <kd>${wheel_kd_gazebo}</kd>
+    <maxContacts>${wheel_max_contacts_gazebo}</maxContacts>
   </gazebo>
 </robot>

File: ROS2_foxy/wheebbot_ws/src/wheebbot/description/urdf/wheebbot.urdf (robot description, URDF)
Before this commit: robot wheebbot, 4 links, 3 joints
Links:
- removed link base_link
- added link aux_link
- link left_wheel: geometry collision cylinder length=0.02 radius=0.06; visual mesh filename=package://wheebbot/description/meshes/wheel_black.dae scale=1.0 1.0 1.0
- link right_wheel: geometry collision cylinder length=0.02 radius=0.06; visual mesh filename=package://wheebbot/description/meshes/wheel_black.dae scale=1.0 1.0 1.0
Joints:
- removed joint floating_base_joint
- added joint aux_joint: type fixed, parent aux_link, child body, origin xyz=0 0 0.43800000000000006 rpy=0 0 0
- joint left_wheel_joint: limit effort=30 velocity=100.0 -> effort=30.0 velocity=100.0
- joint right_wheel_joint: limit effort=30 velocity=100.0 -> effort=30.0 velocity=100.0

File: ROS2_foxy/wheebbot_ws/src/wheebbot/description/urdf/wheebbot.urdf.xacro (robot description, xacro)
@@ -145,6 +145,6 @@
     <child link="left_wheel"/>
     <axis xyz="0 1 0" />
-    <dynamics damping="0.0" friction="0.0"/>
-    <limit effort="30" velocity="100.0" />
+    <dynamics damping="${wheel_joint_damping}" friction="${wheel_joint_static_friction}"/>
+    <limit effort="${wheel_joint_effort_lim}" velocity="${wheel_joint_velocity_lim}" />
   </joint>
   <joint name="right_wheel_joint" type="continuous">
@@ -153,6 +153,6 @@
     <child link="right_wheel"/>
     <axis xyz="0 1 0" />
-    <dynamics damping="0.0" friction="0.0"/>
-    <limit effort="30" velocity="100.0" />
+    <dynamics damping="${wheel_joint_damping}" friction="${wheel_joint_static_friction}"/>
+    <limit effort="${wheel_joint_effort_lim}" velocity="${wheel_joint_velocity_lim}" />
   </joint>
 </robot>
